File: labs/19-pcb/parthiv_pcb/parthiv_pcb.kicad_sch (KiCad schematic)
At the start: 0 parts

Commit message: major
Parts:
- added C1, C2: 10 uF, Capacitor_SMD:CP_Elec_4x5.4, symbol Device:C_Polarized
- added J1: UART, Connector_PinSocket_2.54mm:PinSocket_1x05_P2.54mm_Horizontal, symbol parthiv_pcb:UART
- added J2: Raspberry_Pi_2_3, Connector_PinSocket_2.54mm:PinSocket_2x20_P2.54mm_Vertical, symbol Connector:Raspberry_Pi_2_3
- added U1, U2: NRF24L01_Breakout, RF_Module:nRF24L01_Breakout, symbol RF:NRF24L01_Breakout
Connections:
- new net: J2.31 (GCLK2/GPIO6), U2.3 (CE)
- new net: J2.24 (~{CE0}/GPIO8), U2.4 (~{CSN})
- new net: J2.23 (SCLK0/GPIO11), U1.5 (SCK), U2.5 (SCK)
- new net: J2.19 (MOSI0/GPIO10), U1.6 (MOSI), U2.6 (MOSI)
- new net: J2.21 (MISO0/GPIO9), U1.7 (MISO), U2.7 (MISO)
- new net: J1.2 (TX), J2.10 (GPIO15/RXD)
- new net: J1.3 (RX), J2.8 (GPIO14/TXD)
- new net: J2.29 (GCLK1/GPIO5), U1.3 (CE)
- new net: J2.26 (~{CE1}/GPIO7), U1.4 (~{CSN})
- new net +3V3: C1.1, C2.1, J2.1 (3V3), J2.17 (3V3), U1.2 (VCC), U2.2 (VCC)
- new net +5V: J1.5 (5V), J2.2 (5V), J2.4 (5V)
- new net GND: C1.2, C2.2, J1.4 (GND), J2.14 (GND), J2.20 (GND), J2.25 (GND), J2.30 (GND), J2.34 (GND), J2.39 (GND), J2.6 (GND), J2.9 (GND), U1.1 (GND), U2.1 (GND)
- no-connect marks 0 -> 22
